File: Card/L1IFStream.kicad_pcb (KiCad board)
At the start: 4 copper layers, 156.3 x 127.3 mm, 125 parts, among them J1 Conn_Coaxial, J2 USB_A, J3 RF_Shield_One_Piece, J4 Conn_Coaxial, U1 MAX2769ETI+T, U10 74LVC374, U11 74HC2G04, U2 TPS717285DCKR, U3 TPS717285DCKR, U4 NCP164CSN330T1G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

Commit message: Floof planning USB stick
Parts:
- added REF**: USB_A_CNCTech_1001-011-01101_Horizontal, L1IFStream:USB_A_CNCTech_1001-011-01101_Horizontal, F.Cu at (30.7, 182.7)
- moved U4 49.5 mm to (76.5, 157.4)
- moved U5 49.5 mm to (78.7, 144.0)
- moved X2 49.5 mm to (77.6, 149.1)
- moved U6 32.4 mm to (59.9, 150.4)
Changed lines of the file:
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@@
+        (effects (font (size 1 1) (thickness 0.15)))
+    )
+    (fp_text user "0.132in/3.353mm" (at 0 4.7244 -90) (layer "Dwgs.User")
+        (effects (font (size 1 1) (thickness 0.15)))
+    )
+    (fp_text user "0.038in/0.965mm" (at -2.3749 -5.4229 -90) (layer "Dwgs.User")
+        (effects (font (size 1 1) (thickness 0.15)))
+    )
+    (fp_text user "0.187in/4.75mm" (at 7.9629 0.635 -90) (layer "Dwgs.User")
         (effects (font (size 1 1) (thickness 0.15)))
     )
     (fp_text user "0.132in/3.353mm" (at 4.7244 -0.635 -90) (layer "Dwgs.User")
-        (effects (font (size 1 1) (thickness 0.15)))
-    )
-    (fp_text user "0.132in/3.353mm" (at 0 4.7244 -90) (layer "Dwgs.User")
-        (effects (font (size 1 1) (thickness 0.15)))
-    )
-    (fp_text user "0.187in/4.75mm" (at 7.9629 0.635 -90) (layer "Dwgs.User")
-        (effects (font (size 1 1) (thickness 0.15)))
-    )
-    (fp_text user "0.038in/0.965mm" (at -2.3749 -5.4229 -90) (layer "Dwgs.User")
         (effects (font (size 1 1) (thickness 0.15)))
     )
@@
     )
   )
+  (footprint "L1IFStream:USB_A_CNCTech_1001-011-01101_Horizontal" (layer "F.Cu")
+    (at 30.6666 182.6882 180)
+    (descr "USB type A Plug, Horizontal, http://cnctech.us/pdfs/1001-011-01101.pdf")
+    (tags "USB-A")
+    (attr smd)
+    (fp_text reference "REF**" (at -6.9 -8) (layer "F.SilkS")
+        (effects (font (size 1 1) (thickness 0.15)))
+    )
+    (fp_text value "USB_A_CNCTech_1001-011-01101_Horizontal" (at 0 8) (layer "F.Fab")
+        (effects (font (size 1 1) (thickness 0.15)))
+    )
+    (fp_text user "PCB Edge" (at -4.55 -0.05 90) (layer "Dwgs.User")
+        (effects (font (size 0.6 0.6) (thickness 0.09)))
+    )
+    (fp_text user "${REFERENCE}" (at -6 0 90) (layer "F.Fab")
+        (effects (font (size 1 1) (thickness 0.15)))
+    )
+    (fp_line (start -8.02 -4.4) (end -8.775 -4.4)
+      (stroke (width 0.12) (type solid)) (layer "F.SilkS"))
+    (fp_line (start -8.02 -4.4) (end -8.02 4.4)
+      (stroke (width 0.12) (type solid)) (layer "F.SilkS"))
+    (fp_line (start -4.85 -6.145) (end -3.8 -6.145)
+      (stroke (width 0.12) (type solid)) (layer "F.SilkS"))
+    (fp_line (start -4.85 6.145) (end -3.8 6.145)
+      (stroke (width 0.12) (type solid)) (layer "F.SilkS"))
+    (fp_line (start -3.8 6.025) (end -3.8 -6.025)
+      (stroke (width 0.1) (type solid)) (layer "Dwgs.User"))
+    (fp_line (start -11.4 -4.55) (end -9.15 -4.55)
+      (stroke (width 0.05) (type solid)) (layer "F.CrtYd"))
+    (fp_line (start -11.4 4.55) (end -11.4 -4.55)
+      (stroke (width 0.05) (type solid)) (layer "F.CrtYd"))
+    (fp_line (start -11.4 4.55) (end -9.15 4.55)
+      (stroke (width 0.05) (type solid)) (layer "F.CrtYd"))
+    (fp_line (start -9.15 -7.15) (end -9.15 -4.55)
+      (stroke (width 0.05) (type solid)) (layer "F.CrtYd"))
+    (fp_line (start -9.15 -7.15) (end -4.65 -7.15)
+      (stroke (width 0.05) (type solid)) (layer "F.CrtYd"))
+    (fp_line (start -9.15 4.55) (end -9.15 7.15)
+      (stroke (width 0.05) (type solid)) (layer "F.CrtYd"))
+    (fp_line (start -9.15 7.15) (end -4.65 7.15)
+      (stroke (width 0.05) (type solid)) (layer "F.CrtYd"))
+    (fp_line (start -4.65 -6.52) (end -4.65 -7.15)
+      (stroke (width 0.05) (type solid)) (layer "F.CrtYd"))
+    (fp_line (start -4.65 -6.52) (end 11.4 -6.52)
+      (stroke (width 0.05) (type solid)) (layer "F.CrtYd"))
+    (fp_line (start -4.65 6.52) (end 11.4 6.52)
+      (stroke (width 0.05) (type solid)) (layer "F.CrtYd"))
+    (fp_line (start -4.65 7.15) (end -4.65 6.52)
+      (stroke (width 0.05) (type solid)) (layer "F.CrtYd"))
+    (fp_line (start 11.4 6.52) (end 11.4 -6.52)
+      (stroke (width 0.05) (type solid)) (layer "F.CrtYd"))
+    (fp_line (start -10.4 -3.75) (end -7.9 -3.75)
+      (stroke (width 0.1) (type solid)) (layer "F.Fab"))
+    (fp_line (start -10.4 -3.25) (end -10.4 -3.75)
+      (stroke (width 0.1) (type solid)) (layer "F.Fab"))
+    (fp_line (start -10.4 -3.25) (end -7.9 -3.25)
+      (stroke (width 0.1) (type solid)) (layer "F.Fab"))
+    (fp_line (start -10.4 -1.25) (end -7.9 -1.25)
+      (stroke (width 0.1) (type solid)) (layer "F.Fab"))
+    (fp_line (start -10.4 -0.75) (end -10.4 -1.25)
+      (stroke (width 0.1) (type solid)) (layer "F.Fab"))
+    (fp_line (start -10.4 -0.75) (end -7.9 -0.75)
+      (stroke (width 0.1) (type solid)) (layer "F.Fab"))
+    (fp_line (start -10.4 0.75) (end -7.9 0.75)
+      (stroke (width 0.1) (type solid)) (layer "F.Fab"))
+    (fp_line (start -10.4 1.25) (end -10.4 0.75)
+      (stroke (width 0.1) (type solid)) (layer "F.Fab"))
+    (fp_line (start -10.4 1.25) (end -7.9 1.25)
+      (stroke (width 0.1) (type solid)) (layer "F.Fab"))
+    (fp_line (start -10.4 3.25) (end -7.9 3.25)
+      (stroke (width 0.1) (type solid)) (layer "F.Fab"))
+    (fp_line (start -10.4 3.75) (end -10.4 3.25)
+      (stroke (width 0.1) (type solid)) (layer "F.Fab"))
+    (fp_line (start -10.4 3.75) (end -7.9 3.75)
+      (stroke (width 0.1) (type solid)) (layer "F.Fab"))
+    (fp_line (start -7.9 -6.025) (end 10.9 -6.025)
+      (stroke (width 0.1) (type solid)) (layer "F.Fab"))
+    (fp_line (start -7.9 6.025) (end -7.9 -6.025)
+      (stroke (width 0.1) (type solid)) (layer "F.Fab"))
+    (fp_line (start -7.9 6.025) (end 10.9 6.025)
+      (stroke (width 0.1) (type solid)) (layer "F.Fab"))
+    (fp_line (start -7.75 -3.5) (end -7.25 -4)
+      (stroke (width 0.1) (type solid)) (layer "F.Fab"))
+    (fp_line (start -7.75 -3.5) (end -7.25 -3)
+      (stroke (width 0.1) (type solid)) (layer "F.Fab"))
+    (fp_line (start -7.25 -4) (end -7.25 -3.05)
+      (stroke (width 0.1) (type solid)) (layer "F.Fab"))
+    (fp_line (start 10.9 6.025) (end 10.9 -6.025)
+      (stroke (width 0.1) (type solid)) (layer "F.Fab"))
+    (fp_circle (center -6.9 -2.3) (end -6.9 -2.8)
+      (stroke (width 0.1) (type solid)) (fill none) (layer "F.Fab"))
+    (fp_circle (center -6.9 2.3) (end -6.9 2.8)
+      (stroke (width 0.1) (type solid)) (fill none) (layer "F.Fab"))
+    (pad "" np_thru_hole circle (at -6.9 -2.3 180) (size 1.1 1.1) (drill 1.1) (layers "*.Cu" "*.Mask"))
+    (pad "" np_thru_hole circle (at -6.9 2.3 180) (size 1.1 1.1) (drill 1.1) (layers "*.Cu" "*.Mask"))
+    (pad "1" smd rect (at -9.65 -3.5 180) (size 2.5 1.1) (layers "F.Cu" "F.Paste" "F.Mask"))
+    (pad "2" smd rect (at -9.65 -1 180) (size 2.5 1.1) (layers "F.Cu" "F.Paste" "F.Mask"))
+    (pad "3" smd rect (at -9.65 1 180) (size 2.5 1.1) (layers "F.Cu" "F.Paste" "F.Mask"))
+    (pad "4" smd rect (at -9.65 3.5 180) (size 2.5 1.1) (layers "F.Cu" "F.Paste" "F.Mask"))
+    (pad "5" thru_hole oval (at -6.9 -5.7 180) (size 3.5 1.9) (drill oval 2.5 0.9) (layers "*.Cu" "*.Mask"))
+    (pad "5" thru_hole oval (at -6.9 5.7 180) (size 3.5 1.9) (drill oval 2.5 0.9) (layers "*.Cu" "*.Mask"))
+    (model "${KISYS3DMOD}/Connector_USB.3dshapes/USB_A_CNCTech_1001-011-01101_Horizontal.wrl"
+      (offset (xyz 0 0 0))
+      (scale (xyz 1 1 1))
+      (rotate (xyz 0 0 0))
+    )
+  )
   (footprint "L1IFStream:TSOT-23-5" (layer "F.Cu")
-    (at 38.275 188.775 -90)
+    (at 76.5388 157.427401 -90)
     (descr "5-pin TSOT23 package, http://cds.linear.com/docs/en/packaging/SOT_5_05-08-1635.pdf")
     (tags "TSOT-23-5")
@@
   )
   (footprint "L1IFStream:SIT2024BA-S8-33E-12.000000E" (layer "F.Cu")
-    (at 39.325 180.425 -90)
+    (at 77.5888 149.077401 -90)
     (property "Description" "MEMS OSC XO 12.0000MHZ LVCMOS LV")
     (property "Digi-Key" "1473-SIT2024BA-S8-33E-12.000000G-ND")
@@
         (effects (font (size 1 1) (thickness 0.15)))
     )
+    (fp_text user "0.051in/1.3mm" (at -1.25 -4.5085 -90) (layer "Dwgs.User")
+        (effects (font (size 1 1) (thickness 0.15)))
+    )
+    (fp_text user "0.022in/0.55mm" (at 4.298 -0.95 -90) (layer "Dwgs.User")
+        (effects (font (size 1 1) (thickness 0.15)))
+    )
+    (fp_text user "0.037in/0.95mm" (at -4.298 -0.475 -90) (layer "Dwgs.User")
+        (effects (font (size 1 1) (thickness 0.15)))
+    )
     (fp_text user "0.098in/2.5mm" (at 0 3.998 -90) (layer "Dwgs.User")
-        (effects (font (size 1 1) (thickness 0.15)))
-    )
-    (fp_text user "0.051in/1.3mm" (at -1.25 -4.5085 -90) (layer "Dwgs.User")
-        (effects (font (size 1 1) (thickness 0.15)))
-    )
-    (fp_text user "0.037in/0.95mm" (at -4.298 -0.475 -90) (layer "Dwgs.User")
-        (effects (font (size 1 1) (thickness 0.15)))
-    )
-    (fp_text user "0.022in/0.55mm" (at 4.298 -0.95 -90) (layer "Dwgs.User")
         (effects (font (size 1 1) (thickness 0.15)))
     )
@@
   )
   (footprint "L1IFStream:93LC66BT-I&slash_OT" (layer "F.Cu")
-    (at 40.4 175.325)
+    (at 78.6638 143.977401)
     (property "Description" "IC EEPROM 4K SPI 2MHZ SOT23-6")
     (property "Digi-Key" "93LC66BT-I/OTCT-ND")
@@
   )
   (footprint "L1IFStream:LQFP-64_10x10mm_P0.5mm" (layer "F.Cu")
-    (at 50.1 181.325)
+    (at 59.908 150.408)
     (descr "LQFP, 64 Pin (https://www.analog.com/media/en/technical-documentation/data-sheets/ad7606_7606-6_7606-4.pdf), generated with kicad-footprint-generator ipc_gullwing_generator.py")
     (tags "LQFP QFP")
@@
   (gr_line (start 23.402215 188.700571) (end 23.451802 188.7018)
     (stroke (width 0.15) (type solid)) (layer "Edge.Cuts"))
+  (gr_line (start 34.446908 175.740638) (end 34.451802 189.7018)
+    (stroke (width 0.15) (type default)) (layer "Edge.Cuts"))
   (gr_line (start 88.018575 173.600965) (end 88.003243 173.554627)
     (stroke (width 0.15) (type solid)) (layer "Edge.Cuts"))

Commit message: Start looking for smaller parts
Parts:
- removed the U9 at (63.1, 178.7)
- removed the U9 at (63.4, 186.1)
- added REF**: DHVQFN-20-1EP_2.5x4.5mm_P0.5mm_EP1x3mm, Package_DFN_QFN:DHVQFN-20-1EP_2.5x4.5mm_P0.5mm_EP1x3mm, F.Cu at (59.8, 185.3)
- added REF**: QFN-56-1EP_8x8mm_P0.5mm_EP6.1x6.1mm_ThermalVias, Package_DFN_QFN:QFN-56-1EP_8x8mm_P0.5mm_EP6.1x6.1mm_ThermalVias, F.Cu at (49.7, 182.4)
- added REF**: DHVQFN-20-1EP_2.5x4.5mm_P0.5mm_EP1x3mm, Package_DFN_QFN:DHVQFN-20-1EP_2.5x4.5mm_P0.5mm_EP1x3mm, F.Cu at (59.7, 180.1)

Commit message: Some floor planning
Parts:
- removed the X3 at (79.7, 178.0)
- added J4: Conn_Coaxial, L1IFStream:MMCX_Molex_73415-1471_Vertical, F.Cu at (126.0, 184.9)
- added REF**: Laird_Technologies_BMI-S-102_16.50x16.50mm, RF_Shielding:Laird_Technologies_BMI-S-102_16.50x16.50mm, F.Cu at (114.8, 181.9)
- added REF**: QPQ1060_1.4x1.2, L1IFStream:QPQ1060_1.4x1.2, F.Cu at (81.2, 177.3)
- added REF**: QPQ1060_1.4x1.2, L1IFStream:QPQ1060_1.4x1.2, F.Cu at (118.1, 176.6)
- added U1: MAX2769ETI+T, L1IFStream:MAX2769ETI&plus_T, F.Cu at (117.8, 181.9)
- added U2: TPS717285DCKR, L1IFStream:TPS717285DCKR, F.Cu at (109.4, 177.9)
- added U3: TPS717285DCKR, L1IFStream:TPS717285DCKR, F.Cu at (109.5, 182.4)
- added X1: SIT5156, L1IFStream:10L_CQFN, F.Cu at (113.1, 186.9)
- moved U1 0.97 mm to (81.0, 181.7)
Routing:
- net (no net): track 0.00 -> 12.3 mm
